Commit message: Basic Map merge working

File: tortoisebot_description/models/urdf/tortoisebot_simple.xacro (robot description, xacro)
@@ -1,8 +1,9 @@
 <?xml version="1.0" ?>
-<robot name="tortoisebot_simple" xmlns:xacro="http://www.ros.org/wiki/xacro">
+<robot name="$(arg namespace)/tortoisebot_simple" xmlns:xacro="http://www.ros.org/wiki/xacro">
+<xacro:property name="robot_name" value="$(arg namespace)"/>
 <!-- <xacro:include filename="$(find tortoisebot_gazebo)/gazebo/tortoisebot_materials.gazebo" /> -->
 <xacro:include filename="$(find tortoisebot_gazebo)/gazebo/tortoisebot_physics.gazebo" />
 <xacro:include filename="$(find tortoisebot_gazebo)/gazebo/tortoisebot_plugins.gazebo" />
-<link name="base_link">
+<link name="${robot_name}/base_link">
   <inertial>
     <origin xyz="-0.030635608127622015 -0.0004221703596385517 0.07737044666769882" rpy="0 0 0"/>
@@ -23,5 +24,5 @@
   </collision>
 </link>
-<link name="wheel_left">
+<link name="${robot_name}/wheel_left">
   <inertial>
     <origin xyz="-5.817360584857412e-08 0.008992666701213833 -2.8524983942262994e-07" rpy="0 0 0"/>
@@ -42,5 +43,5 @@
   </collision>
 </link>
-<link name="wheel_right">
+<link name="${robot_name}/wheel_right">
   <inertial>
     <origin xyz="1.1651486266691519e-09 -0.008992199795129496 -2.763726826629509e-07" rpy="0 0 0"/>
@@ -61,5 +62,5 @@
   </collision>
 </link>
-<link name="lidar">
+<link name="${robot_name}/lidar">
   <inertial>
     <origin xyz="1.6353780135647256e-10 -1.7329123482757136e-13 0.004356361811340997" rpy="0 0 0"/>
@@ -80,5 +81,5 @@
   </collision>
 </link>
-<link name="camera_link">
+<link name="${robot_name}/camera_link">
   <inertial>
     <origin xyz="0.0005000001639132029 -1.7004031399497072e-07 1.1512051351081354e-07" rpy="0 0 0"/>
@@ -99,5 +100,5 @@
   </collision>
 </link>
-<link name="camera_holder">
+<link name="${robot_name}/camera_holder">
   <inertial>
     <origin xyz="0.012956561190815237 4.623703165912345e-06 0.0017885934065832443" rpy="0 0 0"/>
@@ -118,5 +119,5 @@
   </collision>
 </link>
-<link name="castor_wheel">
+<link name="${robot_name}/castor_wheel">
   <inertial>
     <origin xyz="2.5326962749261384e-14 4.504651888394023e-14 -0.0017582044401419582" rpy="0 0 0"/>
@@ -137,41 +138,41 @@
   </collision>
 </link>
-<link name="imu_link"/>
-<joint name="wheel_left_joint" type="continuous">
+<link name="${robot_name}/imu_link"/>
+<joint name="${robot_name}/wheel_left_joint" type="continuous">
   <origin xyz="-0.000197 0.0778 0.032453" rpy="0 0 0"/>
-  <parent link="base_link"/>
-  <child link="wheel_left"/>
+  <parent link="${robot_name}/base_link"/>
+  <child link="${robot_name}/wheel_left"/>
   <axis xyz="0.0 1.0 0.0"/>
 </joint>
-<joint name="wheel_right_joint" type="continuous">
+<joint name="${robot_name}/wheel_right_joint" type="continuous">
   <origin xyz="0.0001 -0.0778 0.032453" rpy="0 0 0"/>
-  <parent link="base_link"/>
-  <child link="wheel_right"/>
+  <parent link="${robot_name}/base_link"/>
+  <child link="${robot_name}/wheel_right"/>
   <axis xyz="0.0 1.0 0.0"/>
 </joint>
-<joint name="lidar_joint" type="fixed">
+<joint name="${robot_name}/lidar_joint" type="fixed">
   <origin xyz="-0.03275 0.0 0.167" rpy="0 0 0"/>
-  <parent link="base_link"/>
-  <child link="lidar"/>
+  <parent link="${robot_name}/base_link"/>
+  <child link="${robot_name}/lidar"/>
 </joint>
-<joint name="camera_sensor_joint" type="fixed">
+<joint name="${robot_name}/camera_sensor_joint" type="fixed">
   <origin xyz="0.019 1e-05 0.002844" rpy="0 0 0"/>
-  <parent link="camera_holder"/>
-  <child link="camera_link"/>
+  <parent link="${robot_name}/camera_holder"/>
+  <child link="${robot_name}/camera_link"/>
 </joint>
-<joint name="camera_tilt_joint" type="fixed">
+<joint name="${robot_name}/camera_tilt_joint" type="fixed">
   <origin xyz="0.03125 0.0 0.131063" rpy="0 0 0"/>
-  <parent link="base_link"/>
-  <child link="camera_holder"/>
+  <parent link="${robot_name}/base_link"/>
+  <child link="${robot_name}/camera_holder"/>
 </joint>
-<joint name="castor_joint" type="fixed">
+<joint name="${robot_name}/castor_joint" type="fixed">
   <origin xyz="-0.0767 0.0 0.0049" rpy="0 0 0"/>
-  <parent link="base_link"/>
-  <child link="castor_wheel"/>
+  <parent link="${robot_name}/base_link"/>
+  <child link="${robot_name}/castor_wheel"/>
 </joint>
-<joint name="imu_joint" type="fixed">
+<joint name="${robot_name}/imu_joint" type="fixed">
   <origin xyz="0.0 0.0 0.11" rpy="0 0 0"/>
-  <parent link="base_link"/>
-  <child link="imu_link"/>
+  <parent link="${robot_name}/base_link"/>
+  <child link="${robot_name}/imu_link"/>
 </joint>
 </robot>
